File: hardware/system/system.sch (KiCad schematic (older format))
At the start: 20 parts, among them J1 CART_SOCKET_28P, J2 EXT_PINS, SW1 POWER, SW2 RESET, SW3 A, SW4 B, SW5 UP, SW6 DN, SW7 LF, SW8 RT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

Commit message: Initial board layout (needs routing)
Parts:
- C1, C2: value 1 uF -> 1uF
- J2: footprint Connector_PinSocket_2.54mm:PinSocket_1x11_P2.54mm_Horizontal -> system:EXT_PINS
- SW3, SW4, SW5, SW6, SW7, SW8: footprint Button_Switch_THT:SW_PUSH_6mm -> system:SW_PUSH_6mm
- U1: footprint (none) -> system:ADAFRUIT_MICRO_LIPO
- U3: footprint (none) -> system:DIYMORE_2.42_IN_OLED
Connections:
- net at U3.5 (RES): now also J1.2 (Pin_2); no longer J1.12 (Pin_12)
- net at J1.26 (Pin_26): now also SW1.3 (C); no longer SW1.1 (A)
- net CART_CS renamed D9_A9
- net D9_A9: now also J1.12 (Pin_12); no longer J1.2 (Pin_2)
- no-connect marks 6 -> 7
Other:
- moved on the sheet: J2
Changed lines of the file:
@@
 F 0 "SW3" H 7000 4450 50  0000 C CNN
 F 1 "A" H 7150 4450 50  0000 C CNN
-F 2 "Button_Switch_THT:SW_PUSH_6mm" H 7050 4750 50  0001 C CNN
+F 2 "system:SW_PUSH_6mm" H 7050 4750 50  0001 C CNN
 F 3 "~" H 7050 4750 50  0001 C CNN
 	1    7050 4550
@@
 F 0 "SW4" H 7000 4850 50  0000 C CNN
 F 1 "B" H 7150 4850 50  0000 C CNN
-F 2 "Button_Switch_THT:SW_PUSH_6mm" H 7050 5150 50  0001 C CNN
+F 2 "system:SW_PUSH_6mm" H 7050 5150 50  0001 C CNN
 F 3 "~" H 7050 5150 50  0001 C CNN
 	1    7050 4950
@@
 F 0 "SW5" H 5100 1550 50  0000 C CNN
 F 1 "UP" H 4900 1550 50  0000 C CNN
-F 2 "Button_Switch_THT:SW_PUSH_6mm" H 5000 1850 50  0001 C CNN
+F 2 "system:SW_PUSH_6mm" H 5000 1850 50  0001 C CNN
 F 3 "~" H 5000 1850 50  0001 C CNN
 	1    5000 1650
@@
 F 0 "SW7" H 5100 2350 50  0000 C CNN
 F 1 "LF" H 4900 2350 50  0000 C CNN
-F 2 "Button_Switch_THT:SW_PUSH_6mm" H 5000 2650 50  0001 C CNN
+F 2 "system:SW_PUSH_6mm" H 5000 2650 50  0001 C CNN
 F 3 "~" H 5000 2650 50  0001 C CNN
 	1    5000 2450
@@
 F 0 "SW6" H 5100 1950 50  0000 C CNN
 F 1 "DN" H 4900 1950 50  0000 C CNN
-F 2 "Button_Switch_THT:SW_PUSH_6mm" H 5000 2250 50  0001 C CNN
+F 2 "system:SW_PUSH_6mm" H 5000 2250 50  0001 C CNN
 F 3 "~" H 5000 2250 50  0001 C CNN
 	1    5000 2050
@@
 F 0 "SW8" H 5100 2750 50  0000 C CNN
 F 1 "RT" H 4900 2750 50  0000 C CNN
-F 2 "Button_Switch_THT:SW_PUSH_6mm" H 5000 3050 50  0001 C CNN
+F 2 "system:SW_PUSH_6mm" H 5000 3050 50  0001 C CNN
 F 3 "~" H 5000 3050 50  0001 C CNN
 	1    5000 2850
@@
 	3850 3650 4200 3650
 Wire Wire Line
-	4700 3350 5850 3350
-Wire Wire Line
 	5850 3350 5850 3600
 $Comp
@@
 	4200 3550 4200 3650
 Connection ~ 4200 3650
-Wire Wire Line
-	4200 3650 4700 3650
 Wire Wire Line
 	5950 3600 5950 3250
@@
 F 0 "U1" H 2700 5565 50  0000 C CNN
 F 1 "LIPO_CHARGER" H 2700 5474 50  0000 C CNN
-F 2 "" H 2700 5100 50  0001 C CNN
+F 2 "system:ADAFRUIT_MICRO_LIPO" H 2700 5100 50  0001 C CNN
 F 3 "" H 2700 5100 50  0001 C CNN
 	1    2700 5100
@@
 	3050 4250 3350 4250
 Wire Wire Line
-	4850 3450 4850 4150
-Wire Wire Line
 	7500 4950 7500 5000
 Wire Wire Line
@@
 F 0 "U3" H 5100 4900 50  0000 R CNN
 F 1 "SPI_DISPLAY" H 5250 4800 39  0000 R CNN
-F 2 "" H 5100 4550 30  0001 C CNN
+F 2 "system:DIYMORE_2.42_IN_OLED" H 5100 4550 30  0001 C CNN
 F 3 "" H 5100 4550 30  0001 C CNN
 	1    5050 4650
@@
 P 3750 5350
 F 0 "C1" H 3850 5400 50  0000 L CNN
-F 1 "1 uF" H 3850 5300 50  0000 L CNN
+F 1 "1uF" H 3850 5300 50  0000 L CNN
 F 2 "Capacitor_THT:C_Rect_L4.0mm_W2.5mm_P2.50mm" H 3750 5350 50  0001 C CNN
 F 3 "~" H 3750 5350 50  0001 C CNN
@@
 P 4350 5350
 F 0 "C2" H 4550 5400 50  0000 R CNN
-F 1 "1 uF" H 4650 5300 50  0000 R CNN
+F 1 "1uF" H 4650 5300 50  0000 R CNN
 F 2 "Capacitor_THT:C_Rect_L4.0mm_W2.5mm_P2.50mm" H 4350 5350 50  0001 C CNN
 F 3 "~" H 4350 5350 50  0001 C CNN
@@
 	6150 5350 7200 5350
 Wire Wire Line
-	3750 4150 4850 4150
-Wire Wire Line
 	5350 4850 5450 4850
 Wire Wire Line
@@
 Text GLabel 6550 3450 1    39   Input ~ 0
 MISO
-Text GLabel 5550 4250 3    39   Input ~ 0
-CART_CS
-Wire Wire Line
-	5550 4100 5550 4250
+Wire Wire Line
+	5550 4100 5550 5100
 Wire Wire Line
 	5850 4100 5850 4250
@@
 Text GLabel 5950 4250 3    39   Input ~ 0
 SCL
-Wire Wire Line
-	6550 5050 5150 5050
-Wire Wire Line
-	6550 4100 6550 5050
-Wire Wire Line
-	5150 4850 5150 5050
 Text GLabel 6750 3450 1    39   Input ~ 0
 D10_A10
@@
 L Connector:Conn_01x10_Female J2
 U 1 1 6029D390
-P 8350 3450
-F 0 "J2" V 8515 3380 50  0000 C CNN
-F 1 "EXT_PINS" V 8424 3380 50  0000 C CNN
-F 2 "Connector_PinSocket_2.54mm:PinSocket_1x11_P2.54mm_Horizontal" H 8350 3450 50  0001 C CNN
-F 3 "~" H 8350 3450 50  0001 C CNN
-	1    8350 3450
+P 8250 3450
+F 0 "J2" V 8415 3380 50  0000 C CNN
+F 1 "EXT_PINS" V 8324 3380 50  0000 C CNN
+F 2 "system:EXT_PINS" H 8250 3450 50  0001 C CNN
+F 3 "~" H 8250 3450 50  0001 C CNN
+	1    8250 3450
 	0    -1   -1   0
 $EndComp
@@
 L power:GND #PWR0110
 U 1 1 602A3E9B
+P 7850 3650
+F 0 "#PWR0110" H 7850 3400 50  0001 C CNN
+F 1 "GND" H 7800 3500 50  0000 C CNN
+F 2 "" H 7850 3650 50  0001 C CNN
+F 3 "" H 7850 3650 50  0001 C CNN
+	1    7850 3650
+	1    0    0    -1
+$EndComp
+$Comp
+L power:VCC #PWR0111
+U 1 1 602A5101
 P 7950 3650
-F 0 "#PWR0110" H 7950 3400 50  0001 C CNN
-F 1 "GND" H 7900 3500 50  0000 C CNN
+F 0 "#PWR0111" H 7950 3500 50  0001 C CNN
+F 1 "VCC" V 7950 3800 50  0000 L CNN
 F 2 "" H 7950 3650 50  0001 C CNN
 F 3 "" H 7950 3650 50  0001 C CNN
 	1    7950 3650
-	1    0    0    -1
-$EndComp
-$Comp
-L power:VCC #PWR0111
-U 1 1 602A5101
-P 8050 3650
-F 0 "#PWR0111" H 8050 3500 50  0001 C CNN
-F 1 "VCC" V 8050 3800 50  0000 L CNN
-F 2 "" H 8050 3650 50  0001 C CNN
-F 3 "" H 8050 3650 50  0001 C CNN
-	1    8050 3650
 	1    0    0    1
 $EndComp
 Text GLabel 4850 5200 2    39   Input ~ 0
 3V3
+Text GLabel 8050 3650 3    39   Input ~ 0
+3V3
 Text GLabel 8150 3650 3    39   Input ~ 0
-3V3
+SDA
 Text GLabel 8250 3650 3    39   Input ~ 0
-SDA
+SCL
 Text GLabel 8350 3650 3    39   Input ~ 0
-SCL
+MISO
 Text GLabel 8450 3650 3    39   Input ~ 0
-MISO
+MOSI
 Text GLabel 8550 3650 3    39   Input ~ 0
-MOSI
-Text GLabel 8650 3650 3    39   Input ~ 0
 SCK
 Text GLabel 8750 3650 3    39   Input ~ 0
-CART_CS
-Text GLabel 8850 3650 3    39   Input ~ 0
 D10_A10
+Text GLabel 8650 3650 3    39   Input ~ 0
+D9_A9
+Text GLabel 6550 4250 3    39   Input ~ 0
+D9_A9
+Wire Wire Line
+	6550 4100 6550 4250
+Wire Wire Line
+	4700 3350 5850 3350
+Wire Wire Line
+	5150 4850 5150 5100
+NoConn ~ 3750 4150
+Wire Wire Line
+	4200 3650 4700 3650
+Wire Wire Line
+	5150 5100 5550 5100
+Wire Wire Line
+	4850 4350 3750 4350
+Wire Wire Line
+	4850 3450 4850 4350
 $EndSCHEMATC
