File: hardware/system/system_advance.kicad_pcb (KiCad board)
At the start: 2 copper layers, 528.9 x 87.2 mm, 46 parts, among them J1 CART_SOCKET_28P, J2 EXTENSION PINS, SW1 POWER, SW2 RESET, SW3 A, SW4 B, SW5 UP, SW6 DN, SW7 LF, SW8 RT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

Commit message: wip; layout adjustment
Parts:
- removed C1, C2: 1uF, Capacitor_THT:C_Rect_L4.0mm_W2.5mm_P2.50mm
- removed the HOLE at (103.0, 70.2)
- removed the U2 at (184.7, 78.0)
- J2: value EXTENSION PINS -> EXT_PINS
- moved SW2 103.4 mm to (165.4, 118.7), turned to 0 degrees
- moved R1 96.7 mm to (163.8, 112.6), turned to 0 degrees
- moved **REF 93.0 mm to (113.3, 71.9), turned to 90 degrees
- moved U1 87.9 mm to (108.1, 77.5), turned to 0 degrees
- moved J2 8.44 mm to (138.2, 127.0)
- moved HOLE 8.40 mm to (184.3, 73.0)
- renumbered U3 to U2
Connections:
- J2 pad 10: D9_A9 -> D10_A10
- J2 pad 4: 3V3 -> SDA
- J2 pad 5: SDA -> SCL
- J2 pad 6: SCL -> MISO
- J2 pad 7: MISO -> MOSI
- J2 pad 8: MOSI -> SCK
- J2 pad 9: SCK -> D9_A9
- U2 pad 2: 3V3 -> VCC
Other:
- outline, holes or cut-outs redrawn

Commit message: wip; save
Parts:
- moved REF** 11.7 mm to (178.6, 142.9), turned to 90 degrees
- moved REF** 4.19 mm to (188.3, 145.4), turned to 90 degrees
Other:
- outline, holes or cut-outs redrawn

Commit message: wip; layout (needs routing)
Parts:
- added HOLE: MountingHole_2.7mm_M2.5_Pad, MountingHole:MountingHole_2.7mm_M2.5_Pad, B.Cu at (95.1, 73.0)
- J2: value EXT_PINS -> EXTENSION PINS
- SW1: footprint system:SPDT_SWITCH -> system:SPDT_SWITCH_ADV
- moved **REF 63.0 mm to (176.3, 71.8)
- moved U1 63.0 mm to (171.1, 77.3)
- moved J2 8.39 mm to (139.7, 118.7)
- moved SW7 1.37 mm to (85.9, 92.5)
- moved SW5 1.37 mm to (93.0, 85.3)
- moved SW6 1.37 mm to (93.0, 99.6)
- moved SW8 1.37 mm to (100.1, 92.5)
- moved D1 1.02 mm to (97.8, 111.5)
- moved SW1 0.89 mm to (112.5, 119.0)
- moved R1 0.25 mm to (163.8, 112.9)
- moved SW2 0.25 mm to (165.4, 119.0)
Other:
- outline, holes or cut-outs redrawn
- board text added: "V1.0-dev0"
- board text added: "github.com/menehune23/arduboy-dotmg"
- board text removed: "V1.0-dev5"
